File: DaveJonesTandy1000Turbo/DaveJonesTandy1000Turbo.kicad_pcb (KiCad board)
At the start: 2 copper layers, 12.7 x 100.3 mm, 12 parts, among them CN1 8284 Socket, J1 TO BUS CLOCK, SW1 ON = TURBO, U1 74LS175, U2 74LS86, U3 8284, Y1 20/22MHz Crystal

Commit message: Update to DaveJonesTurbo pcb
Routing:
- net Net-(CN1-Pad2): track 35.1 -> 39.5 mm
- net GND: track 5.08 -> 7.62 mm
Other:
- board size 12.7 x 100.3 mm -> 12.7 x 99.7 mm
