File: CoCoProtoBoard/CoCoProtoBoard.sch (KiCad schematic (older format))
At the start: 6 parts, among them P1 CocoEdgeConnector, P10 Power Bus, P2 Coco Data, P3 Coco Address, P4 Coco Signals

Commit message: CocoProtoBoard: Swap +5v and GND rails and other minor tweaks.
Connections:
- net +5V: now also P10.2 (Pin_2); no longer P10.1 (Pin_1)
- net GND: now also P10.1 (Pin_1); no longer P10.2 (Pin_2)
Changed lines of the file:
@@
 Comment4 ""
 $EndDescr
-$Comp
-L CoCoProtoBoard-rescue:GND #PWR01
-U 1 1 572D1809
-P 1300 4950
-F 0 "#PWR01" H 1300 4700 50  0001 C CNN
-F 1 "GND" H 1300 4800 50  0000 C CNN
-F 2 "" H 1300 4950 50  0000 C CNN
-F 3 "" H 1300 4950 50  0000 C CNN
-	1    1300 4950
-	1    0    0    -1
-$EndComp
 NoConn ~ 1200 900
 NoConn ~ 1200 1000
-$Comp
-L CoCoProtoBoard-rescue:GND #PWR02
-U 1 1 572D77AD
-P 7950 1750
-F 0 "#PWR02" H 7950 1500 50  0001 C CNN
-F 1 "GND" H 7950 1600 50  0000 C CNN
-F 2 "" H 7950 1750 50  0000 C CNN
-F 3 "" H 7950 1750 50  0000 C CNN
-	1    7950 1750
-	1    0    0    -1
-$EndComp
 $Comp
 L Device:CP C1
@@
 L Connector_Generic:Conn_01x02 P10
 U 1 1 57C5B26B
-P 8750 1450
-F 0 "P10" H 8750 1750 50  0000 C CNN
-F 1 "Power Bus" V 8850 1450 50  0000 C CNN
-F 2 "Housings_DIP:DIP-16_W7.62mm" H 8750 250 50  0001 C CNN
-F 3 "" H 8750 250 50  0000 C CNN
-	1    8750 1450
-	1    0    0    -1
-$EndComp
-$Comp
-L CoCoProtoBoard-rescue:GND #PWR07
-U 1 1 57C5B277
-P 8450 1750
-F 0 "#PWR07" H 8450 1500 50  0001 C CNN
-F 1 "GND" H 8450 1600 50  0000 C CNN
-F 2 "" H 8450 1750 50  0000 C CNN
-F 3 "" H 8450 1750 50  0000 C CNN
-	1    8450 1750
-	1    0    0    -1
+P 8750 1550
+F 0 "P10" H 8750 1850 50  0000 C CNN
+F 1 "Power Bus" V 8850 1550 50  0000 C CNN
+F 2 "Housings_DIP:DIP-16_W7.62mm" H 8750 350 50  0001 C CNN
+F 3 "" H 8750 350 50  0000 C CNN
+	1    8750 1550
+	1    0    0    1
 $EndComp
 Wire Wire Line
@@
 	1    0    0    -1
 $EndComp
+$Comp
+L power:GND #PWR?
+U 1 1 60302C76
+P 7950 1750
+F 0 "#PWR?" H 7950 1500 50  0001 C CNN
+F 1 "GND" H 7955 1577 50  0000 C CNN
+F 2 "" H 7950 1750 50  0001 C CNN
+F 3 "" H 7950 1750 50  0001 C CNN
+	1    7950 1750
+	1    0    0    -1
+$EndComp
+$Comp
+L power:GND #PWR?
+U 1 1 6030625B
+P 8450 1750
+F 0 "#PWR?" H 8450 1500 50  0001 C CNN
+F 1 "GND" H 8455 1577 50  0000 C CNN
+F 2 "" H 8450 1750 50  0001 C CNN
+F 3 "" H 8450 1750 50  0001 C CNN
+	1    8450 1750
+	1    0    0    -1
+$EndComp
+$Comp
+L power:GND #PWR?
+U 1 1 60309B34
+P 1300 4950
+F 0 "#PWR?" H 1300 4700 50  0001 C CNN
+F 1 "GND" H 1305 4777 50  0000 C CNN
+F 2 "" H 1300 4950 50  0001 C CNN
+F 3 "" H 1300 4950 50  0001 C CNN
+	1    1300 4950
+	1    0    0    -1
+$EndComp
